File: pcb/pcb.kicad_sch (KiCad schematic)
At the start: 203 parts, among them J2 Conn_01x04_Pin, J4 Conn_01x04_Socket, J5 Conn_01x02_Pin, Q1 BSS84, SW1 SW_Push, SW10(8)1 SW_Push_45deg, SW11(9)1 SW_Push_45deg, SW12(0)1 SW_Push_45deg, SW13(-)1 SW_Push_45deg, SW14(=)1 SW_Push_45deg, SW15(bckspc)1 SW_Push_45deg, SW16(tab)1 SW_Push_45deg, SW17(q)1 SW_Push_45deg, SW18(w)1 SW_Push_45deg, SW19(e)1 SW_Push_45deg, SW2 SW_Push, SW2(esc)1 SW_Push_45deg, SW20(r)1 SW_Push_45deg, SW21(t)1 SW_Push_45deg, SW22(y)1 SW_Push_45deg, SW23(u)1 SW_Push_45deg, SW24(i)1 SW_Push_45deg, SW25(o)1 SW_Push_45deg, SW26(p)1 SW_Push_45deg, SW27([)1 SW_Push_45deg, SW28(])1 SW_Push_45deg, SW29(\)1 SW_Push_45deg, SW3 SW_Push, SW3(1)1 SW_Push_45deg, SW30(caps)1 SW_Push_45deg, SW31(unused)1 SW_Push_45deg, SW32(a)1 SW_Push_45deg, SW33(lshift)1 SW_Push_45deg, SW34(s)1 SW_Push_45deg, SW35(z)1 SW_Push_45deg, SW36(d)1 SW_Push_45deg, SW37(x)1 SW_Push_45deg, SW38(f)1 SW_Push_45deg, SW39(c)1 SW_Push_45deg, SW4 SW_Push, SW4(2)1 SW_Push_45deg, SW40(g)1 SW_Push_45deg, SW41(v)1 SW_Push_45deg, SW42(h)1 SW_Push_45deg, SW43(b)1 SW_Push_45deg, SW44(j)1 SW_Push_45deg, SW45(n)1 SW_Push_45deg, SW46(k)1 SW_Push_45deg, SW47(m)1 SW_Push_45deg, SW48(l)1 SW_Push_45deg, SW49(,)1 SW_Push_45deg, SW5(3)1 SW_Push_45deg, SW50(;)1 SW_Push_45deg, SW51(.)1 SW_Push_45deg, SW52(')1 SW_Push_45deg, SW53(/)1 SW_Push_45deg, SW54(ret)1 SW_Push_45deg, SW55(rshift)1 SW_Push_45deg, SW56(unused)1 SW_Push_45deg, SW57(up)1 SW_Push_45deg, SW58(globe)1 SW_Push_45deg, SW6(4)1 SW_Push_45deg, SW60(lctrl)1 SW_Push_45deg, SW62(super)1 SW_Push_45deg, SW64(lalt)1 SW_Push_45deg, SW66(spc)1 SW_Push_45deg, SW68(spc)1 SW_Push_45deg, SW7(5)1 SW_Push_45deg, SW70(spc)1 SW_Push_45deg, SW72(spc)1 SW_Push_45deg, SW74(spc)1 SW_Push_45deg, SW76(ralt)1 SW_Push_45deg, SW78(rctrl)1 SW_Push_45deg, SW8(6)1 SW_Push_45deg, SW80(left)1 SW_Push_45deg, SW82(down)1 SW_Push_45deg, SW84(right)1 SW_Push_45deg, SW9(7)1 SW_Push_45deg, U1 ESP32-C3-WROOM-02, U2 AP2112K-3.3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

Commit message: add stuff
Parts:
- removed C6: 2.2uF, Capacitor_SMD:C_0603_1608Metric_Pad1.08x0.95mm_HandSolder, symbol Device:C
- removed C7: 100nF, Capacitor_SMD:C_0603_1608Metric_Pad1.08x0.95mm_HandSolder, symbol Device:C
- added Q2, Q3: BSS84, Package_TO_SOT_SMD:SOT-23, symbol Transistor_FET:BSS84
- added R33, R34: 100k, Resistor_SMD:R_1206_3216Metric_Pad1.30x1.75mm_HandSolder, symbol Device:R
- added SW5: RS601A-1020013BB, easyeda2kicad:SW-TH_RS601A-1020013BB, symbol easyeda2kicad:RS601A-1020013BB
- added U6: BH-AAA-B5AA005, easyeda2kicad:BH-AAA-B5AA005, symbol easyeda2kicad:BH-AAA-B5AA005
Connections:
- net GND: now also R33.2, R34.2, U6.1 (-)
- net VBUS: now also Q2.3 (D), Q3.3 (D), SW5.2; no longer C1.1, U2.1 (VIN), U2.3 (EN), USB1.11 (VBUS), USB1.2 (VBUS)
- new net: C1.1, SW5.1, U2.1 (VIN), U2.3 (EN)
- new net: Q2.1 (G), R33.1
- new net: Q3.1 (G), R34.1
- new net: U6.2 (+), U6.3 (-)
- new net: U6.5 (-), U6.6 (+)
- new net B+: Q2.2 (S), U6.4 (+)
- new net USB_VBUS: Q3.2 (S), USB1.11 (VBUS), USB1.2 (VBUS)

Commit message: stuff
Parts:
- R1, R2, R31: footprint Resistor_SMD:R_1206_3216Metric_Pad1.30x1.75mm_HandSolder -> Resistor_SMD:R_0603_1608Metric
- R19, R20, R21, R22, R23, R24, R25, R3, R32, R4: footprint Resistor_SMD:R_1206_3216Metric_Pad1.30x1.75mm_HandSolder -> Resistor_SMD:R_0805_2012Metric
- R27, R28, R29: value 45k -> 47k; footprint Resistor_SMD:R_1206_3216Metric_Pad1.30x1.75mm_HandSolder -> Resistor_SMD:R_0402_1005Metric
Changed lines of the file:
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@@
 			)
 		)
-		(property "Footprint" "Resistor_SMD:R_1206_3216Metric_Pad1.30x1.75mm_HandSolder"
+		(property "Footprint" "Resistor_SMD:R_0805_2012Metric"
 			(at 25.908 43.18 90)
 			(effects
@@
 			)
 		)
-		(property "Footprint" "Resistor_SMD:R_1206_3216Metric_Pad1.30x1.75mm_HandSolder"
+		(property "Footprint" "Resistor_SMD:R_0805_2012Metric"
 			(at 416.56 290.068 90)
 			(effects
@@
 			)
 		)
-		(property "Footprint" "Resistor_SMD:R_1206_3216Metric_Pad1.30x1.75mm_HandSolder"
+		(property "Footprint" "Resistor_SMD:R_0603_1608Metric"
 			(at 205.74 62.992 90)
 			(effects
@@
 			)
 		)
-		(property "Footprint" "Resistor_SMD:R_1206_3216Metric_Pad1.30x1.75mm_HandSolder"
+		(property "Footprint" "Resistor_SMD:R_0603_1608Metric"
 			(at 204.47 47.752 90)
 			(effects
@@
 			)
 		)
-		(property "Footprint" "Resistor_SMD:R_1206_3216Metric_Pad1.30x1.75mm_HandSolder"
+		(property "Footprint" "Resistor_SMD:R_0805_2012Metric"
 			(at 55.118 60.96 90)
 			(effects
@@
 			)
 		)
-		(property "Footprint" "Resistor_SMD:R_1206_3216Metric_Pad1.30x1.75mm_HandSolder"
+		(property "Footprint" "Resistor_SMD:R_0805_2012Metric"
 			(at 416.56 309.118 90)
 			(effects
@@
 			)
 		)
-		(property "Footprint" "Resistor_SMD:R_1206_3216Metric_Pad1.30x1.75mm_HandSolder"
+		(property "Footprint" "Resistor_SMD:R_0603_1608Metric"
 			(at 521.462 128.27 90)
 			(effects
@@
 			)
 		)
-		(property "Footprint" "Resistor_SMD:R_1206_3216Metric_Pad1.30x1.75mm_HandSolder"
+		(property "Footprint" "Resistor_SMD:R_0805_2012Metric"
 			(at 535.432 128.27 90)
 			(effects
@@
 			)
 		)
-		(property "Footprint" "Resistor_SMD:R_1206_3216Metric_Pad1.30x1.75mm_HandSolder"
+		(property "Footprint" "Resistor_SMD:R_0805_2012Metric"
 			(at 416.56 251.968 90)
 			(effects
@@
 			)
 		)
-		(property "Value" "45k"
+		(property "Value" "47k"
 			(at 128.27 166.3699 0)
 			(effects
@@
 			)
 		)
-		(property "Footprint" "Resistor_SMD:R_1206_3216Metric_Pad1.30x1.75mm_HandSolder"
+		(property "Footprint" "Resistor_SMD:R_0402_1005Metric"
 			(at 129.032 165.1 90)
 			(effects
@@
 			)
 		)
-		(property "Footprint" "Resistor_SMD:R_1206_3216Metric_Pad1.30x1.75mm_HandSolder"
+		(property "Footprint" "Resistor_SMD:R_0805_2012Metric"
 			(at 416.56 328.168 90)
 			(effects
@@
 			)
 		)
-		(property "Value" "45k"
+		(property "Value" "47k"
 			(at 113.03 166.3699 0)
 			(effects
@@
 			)
 		)
-		(property "Footprint" "Resistor_SMD:R_1206_3216Metric_Pad1.30x1.75mm_HandSolder"
+		(property "Footprint" "Resistor_SMD:R_0402_1005Metric"
 			(at 113.792 165.1 90)
 			(effects
@@
 			)
 		)
-		(property "Footprint" "Resistor_SMD:R_1206_3216Metric_Pad1.30x1.75mm_HandSolder"
+		(property "Footprint" "Resistor_SMD:R_0805_2012Metric"
 			(at 47.498 60.96 90)
 			(effects
@@
 			)
 		)
-		(property "Value" "45k"
+		(property "Value" "47k"
 			(at 120.65 166.3699 0)
 			(effects
@@
 			)
 		)
-		(property "Footprint" "Resistor_SMD:R_1206_3216Metric_Pad1.30x1.75mm_HandSolder"
+		(property "Footprint" "Resistor_SMD:R_0402_1005Metric"
 			(at 121.412 165.1 90)
 			(effects
@@
 			)
 		)
-		(property "Footprint" "Resistor_SMD:R_1206_3216Metric_Pad1.30x1.75mm_HandSolder"
+		(property "Footprint" "Resistor_SMD:R_0805_2012Metric"
 			(at 416.56 271.018 90)
 			(effects
@@
 			)
 		)
-		(property "Footprint" "Resistor_SMD:R_1206_3216Metric_Pad1.30x1.75mm_HandSolder"
+		(property "Footprint" "Resistor_SMD:R_0805_2012Metric"
 			(at 38.608 60.96 90)
 			(effects

Commit message: remove entire trackpad and replace with attatchement for hat (modified from the peacock)
Parts:
- removed C10, C13, C14, C16: 2.2uF, Capacitor_SMD:C_0603_1608Metric_Pad1.08x0.95mm_HandSolder, symbol Device:C
- removed C11, C12, C15, C17: 22nF, Capacitor_SMD:C_0603_1608Metric_Pad1.08x0.95mm_HandSolder, symbol Device:C
- removed C8: 10nF, Capacitor_SMD:C_0603_1608Metric_Pad1.08x0.95mm_HandSolder, symbol Device:C
- removed C9: 100nF, Capacitor_SMD:C_0603_1608Metric_Pad1.08x0.95mm_HandSolder, symbol Device:C
- removed R30: 100k, Resistor_SMD:R_1206_3216Metric_Pad1.30x1.75mm_HandSolder, symbol Device:R
- removed R31: 3.3k, Resistor_SMD:R_0603_1608Metric, symbol Device:R
- removed R32: 10k, Resistor_SMD:R_0805_2012Metric, symbol Device:R
- removed U5: ~, footprints:UFBGA136_MCH-M, symbol 2025-08-11_22-50-31:The_Touch_IC
- added Q5: BSS84, Package_TO_SOT_SMD:SOT-23, symbol Transistor_FET:BSS84
- added R31: 1M, Resistor_SMD:R_1206_3216Metric_Pad1.30x1.75mm_HandSolder, symbol Device:R_Small
Connections:
- net +3.3V: now also Q5.2 (S), R31.1
- net at C5.1, U4.10 (VDD), U4.6 (VDD/NC): now also Q5.3 (D)
- net HARD_OFF_SWITCH: now reaches U1.5 (IO6)
- net HARD_OFF_SWITCH: now also Q5.1 (G), R31.2
- net INT_TOUCH: now reaches U3.18 (P21)
- no-connect marks 1 -> 0
Other:
- note removed: "ATMXT1664T3-CCUR035"
- moved on the sheet: R24, R3, R4
