File: pcb/pcb.kicad_pcb (KiCad board)
At the start: 2 copper layers, 511.6 x 118.1 mm, 201 parts, among them J2 Conn_01x04_Pin, J4 Conn_01x04_Socket, J5 Conn_01x02_Pin, J8 Conn_01x08_Pin, Q1 BSS84, Q2 BSS84, Q3 BSS84, Q5 BSS84, SW1 SW_Push, SW10(8)1 SW_Push_45deg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

Commit message: make a hat attatchement
Routing:
- net B-: track 1191.3 -> 1194.1 mm
- net Net-(U3-P20): track 366.2 -> 367.0 mm
Other:
- board size 511.6 x 118.1 mm -> 511.6 x 117.8 mm
